File: PCBs/Didactic_main_PCB/Didactic_main_PCB.kicad_pcb (KiCad board)
At the start: 4 copper layers, 124 x 100 mm, 257 parts, among them IC201 NXB0108PWJ, IC202 NXB0108PWJ, IC601 NXB0108PWJ, IC602 NXB0108PWJ, IC701 AP7179DSKZ20-13, IC702 AP7179DSKZ20-13, J201 Conn_02x08_Odd_Even, J202 Conn_02x08_Odd_Even, J203 Conn_01x02_Pin, J204 Conn_02x18_Odd_Even, J206 10067847-001RLF, J301 690-005-299-043, J401 Conn_01x04_Pin, J402 Conn_01x04_Pin, J403 Conn_ARM_SWD_TagConnect_TC2030, J404 690-005-299-043, J405 Conn_01x04_Pin, J501 PJ-036AH-SMT-TR, J601 Conn_02x08_Odd_Even, J603 Conn_02x08_Odd_Even, J604 SSW-106-02-T-D-RA, J605 SSW-106-02-T-D-RA, U202 SI5351A-B-GT, U301 USBLC6-2SC6, U302 SN74AVC4T774PWR, U303 SN74AVC4T774PWR, U304 FT2232HQ, U305 93LC56BT_SN, U401 STM32G431CBT6, U402 USBLC6-2SC6, U403 INA4180A4IPWR, U501 TPS564255DRLR, U701 TPS7A4533KTTR, Y201 ECS-250-8-33B-CKM-TR, Y301 ECS-120-8-33-JGN-TR3, Y401 ECS-250-8-33B-CKM-TR

Commit message: fixed 3V3 IO EN silkscreen and changed STATUS led to green
Changed lines of the file:
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@@
 	)
 	(gr_text "0"
-		(at 126 135.79 0)
+		(at 135.8 135.8 0)
 		(layer "F.SilkS")
 		(effects
@@
 	)
 	(gr_text "1"
-		(at 135.9 135.78 0)
-		(layer "F.SilkS")
-		(effects
+		(at 126 135.7 0)
+		(layer "F.SilkS")
+		(effects
