File: PCBs/Didactic_main_PCB/PowerMCU.kicad_sch (KiCad schematic)
At the start: 34 parts, among them J401 Conn_01x04_Pin, J402 Conn_01x04_Pin, J403 Conn_ARM_SWD_TagConnect_TC2030, J404 690-005-299-043, J405 Conn_01x04_Pin, U401 STM32G431CBT6, U402 USBLC6-2SC6, U403 INA4180A4IPWR, Y401 ECS-250-8-33B-CKM-TR

Commit message: fixed 3V3 IO EN silkscreen and changed STATUS led to green
Parts:
- D401: MANUFACTURER_PART_NUMBER APHD1608LSURCK -> APHD1608LCGCK
Changed lines of the file:
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@@
 			)
 		)
-		(property "MANUFACTURER_PART_NUMBER" "APHD1608LSURCK "
+		(property "MANUFACTURER_PART_NUMBER" "APHD1608LCGCK"
 			(at 179.07 146.05 0)
 			(effects
